Commit message: fishbot

File: src/caterpillar_robot/urdf/transbot_astra.urdf (robot description, URDF)
Before this commit: robot transbot_description, 12 links, 11 joints
Links:
- link arm: geometry collision mesh filename=file:///home/dillon/UVSIM/src/caterpillar_robot/meshes/arm.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; visual mesh filename=file:///home/dillon/UVSIM/src/caterpillar_robot/meshes/arm.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
- link arm_link1: geometry collision mesh filename=file:///home/dillon/UVSIM/src/caterpillar_robot/meshes/arm_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; visual mesh filename=file:///home/dillon/UVSIM/src/caterpillar_robot/meshes/arm_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
- link arm_link2: geometry collision mesh filename=file:///home/dillon/UVSIM/src/caterpillar_robot/meshes/arm_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; visual mesh filename=file:///home/dillon/UVSIM/src/caterpillar_robot/meshes/arm_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
- link astra_link: geometry collision mesh filename=file:///home/dillon/UVSIM/src/caterpillar_robot/meshes/astr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; visual mesh filename=file:///home/dillon/UVSIM/src/caterpillar_robot/meshes/astr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
- link base_link: geometry collision mesh filename=file:///home/dillon/UVSIM/src/caterpillar_robot/meshes/base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; visual mesh filename=file:///home/dillon/UVSIM/src/caterpillar_robot/meshes/base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
- link left_link1: geometry collision mesh filename=file:///home/dillon/UVSIM/src/caterpillar_robot/meshes/left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; visual mesh filename=file:///home/dillon/UVSIM/src/caterpillar_robot/meshes/left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
- link left_link2: geometry collision mesh filename=file:///home/dillon/UVSIM/src/caterpillar_robot/meshes/left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; visual mesh filename=file:///home/dillon/UVSIM/src/caterpillar_robot/meshes/left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
- link left_link3: geometry collision mesh filename=file:///home/dillon/UVSIM/src/caterpillar_robot/meshes/left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; visual mesh filename=file:///home/dillon/UVSIM/src/caterpillar_robot/meshes/left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
- link right_link1: geometry collision mesh filename=file:///home/dillon/UVSIM/src/caterpillar_robot/meshes/righ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; visual mesh filename=file:///home/dillon/UVSIM/src/caterpillar_robot/meshes/righ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
- link right_link2: geometry collision mesh filename=file:///home/dillon/UVSIM/src/caterpillar_robot/meshes/righ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; visual mesh filename=file:///home/dillon/UVSIM/src/caterpillar_robot/meshes/righ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
- link right_link3: geometry collision mesh filename=file:///home/dillon/UVSIM/src/caterpillar_robot/meshes/righ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; visual mesh filename=file:///home/dillon/UVSIM/src/caterpillar_robot/meshes/righ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
