Commit message: path plan ok!!!

File: src/caterpillar_robot/urdf/caterpillar_robot.xacro.urdf (robot description, URDF)
Before this commit: robot mycar, 31 links, 30 joints
Links:
- link d435_link: geometry collision box size=0.02505 0.09 0.025; visual mesh filename=file:///home/zj/pkg/realsense_ros2_gazebo/install/realsense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
