Commit message: fix model

File: src/caterpillar_robot/urdf/caterpillar_robot.xacro (robot description, xacro)
@@ -21,9 +21,9 @@
                     <cylinder radius="${radius}" length="${length}" />
                 </geometry>
-                <surface>
+                <!-- <surface>
                     <friction>
                         <ode mu="${mu}" mu2="${mu2}"/>
                     </friction>
-                </surface>
+                </surface> -->
             </collision>
             <xacro:default_inertial mass="0.3"/>
@@ -59,5 +59,5 @@
             </material>
         </collision>
-        <xacro:default_inertial mass="0.3"/>
+        <xacro:default_inertial mass="2"/>
     </link>
     <link name="plat_link">
@@ -170,17 +170,21 @@
         <origin xyz="0 0.0 0.06" rpy="0 0 0"/>
     </joint>
-    <xacro:wheel_func wheel_name="left0" xyz="0.14 -0.095 -0.005" rpy="0 0 0" radius="0.0275" length="0.05" mu="1" mu2="1"/>
+    <xacro:wheel_func wheel_name="left_front" xyz="0.14 -0.095 -0.005" rpy="0 0 0" radius="0.0275" length="0.05" mu="1" mu2="1"/>
+    <xacro:wheel_func wheel_name="left0" xyz="0.14 -0.095 -0.05" rpy="0 0 0" radius="0.015" length="0.05" mu="1" mu2="1"/>
     <xacro:wheel_func wheel_name="left1" xyz="0.075 -0.095 -0.05" rpy="0 0 0" radius="0.015" length="0.05" mu="1" mu2="1"/>
     <xacro:wheel_func wheel_name="left2" xyz="0.025 -0.095 -0.05" rpy="0 0 0" radius="0.015" length="0.05" mu="1" mu2="1"/>
     <xacro:wheel_func wheel_name="left3" xyz="-0.025 -0.095 -0.05" rpy="0 0 0" radius="0.015" length="0.05" mu="1" mu2="1"/>
     <xacro:wheel_func wheel_name="left4" xyz="-0.075 -0.095 -0.05" rpy="0 0 0" radius="0.015" length="0.05" mu="1" mu2="1"/>
-    <xacro:wheel_func wheel_name="left5" xyz="-0.125 -0.095 -0.005" rpy="0 0 0" radius="0.0275" length="0.05" mu="1" mu2="1"/>
+    <xacro:wheel_func wheel_name="left5" xyz="-0.125 -0.095 -0.05" rpy="0 0 0" radius="0.015" length="0.05" mu="1" mu2="1"/>
+    <xacro:wheel_func wheel_name="left_back" xyz="-0.125 -0.095 -0.005" rpy="0 0 0" radius="0.0275" length="0.05" mu="1" mu2="1"/>
     <!-- <xacro:wheel_func wheel_name="leftv" xyz="-0.1 -0.15 -0.04" rpy="0 0 0" radius="0.0275" length="0.05" mu="4" mu2="4"/> -->
-    <xacro:wheel_func wheel_name="right0" xyz="0.14 0.095 -0.005" rpy="0 0 0" radius="0.0275" length="0.05" mu="1" mu2="1"/>
+    <xacro:wheel_func wheel_name="right_front" xyz="0.14 0.095 -0.005" rpy="0 0 0" radius="0.0275" length="0.05" mu="1" mu2="1"/>
+    <xacro:wheel_func wheel_name="right0" xyz="0.14 0.095 -0.05" rpy="0 0 0" radius="0.015" length="0.05" mu="1" mu2="1"/>
     <xacro:wheel_func wheel_name="right1" xyz="0.075 0.095 -0.05" rpy="0 0 0" radius="0.015" length="0.05" mu="1" mu2="1"/>
     <xacro:wheel_func wheel_name="right2" xyz="0.025 0.095 -0.05" rpy="0 0 0" radius="0.015" length="0.05" mu="1" mu2="1"/>
     <xacro:wheel_func wheel_name="right3" xyz="-0.025 0.095 -0.05" rpy="0 0 0" radius="0.015" length="0.05" mu="1" mu2="1"/>
     <xacro:wheel_func wheel_name="right4" xyz="-0.075 0.095 -0.05" rpy="0 0 0" radius="0.015" length="0.05" mu="1" mu2="1"/>
-    <xacro:wheel_func wheel_name="right5" xyz="-0.125 0.095 -0.005" rpy="0 0 0" radius="0.0275" length="0.05" mu="1" mu2="1"/>
+    <xacro:wheel_func wheel_name="right5" xyz="-0.125 0.095 -0.05" rpy="0 0 0" radius="0.015" length="0.05" mu="1" mu2="1"/>
+    <xacro:wheel_func wheel_name="right_back" xyz="-0.125 0.095 -0.005" rpy="0 0 0" radius="0.0275" length="0.05" mu="1" mu2="1"/>
     <!-- <xacro:wheel_func wheel_name="rightv" xyz="-0.1 0.15 -0.04" rpy="0 0 0" radius="0.0275" length="0.05" mu="4" mu2="4"/> -->
     <gazebo reference="base_link">
@@ -233,8 +237,8 @@
     <gazebo>
         <plugin name='diff_drive' filename='libgazebo_ros_planar_move.so'>
-            <leftFrontJoint>left1_joint</leftFrontJoint>
-			<rightFrontJoint>right1_joint</rightFrontJoint>
-			<leftRearJoint>left4_joint</leftRearJoint>
-			<rightRearJoint>right4_joint</rightRearJoint>
+            <leftFrontJoint>left0_joint</leftFrontJoint>
+			<rightFrontJoint>right0_joint</rightFrontJoint>
+			<leftRearJoint>left5_joint</leftRearJoint>
+			<rightRearJoint>right5_joint</rightRearJoint>
             <commandTopic>cmd_vel</commandTopic>
 			<odometryTopic>odom</odometryTopic>

File: src/caterpillar_robot/urdf/caterpillar_robot.xacro.urdf (robot description, URDF)
Before this commit: robot mycar, 18 links, 17 joints
Links:
- added link left_back_link, mass 1; collision cylinder length=0.05 radius=0.0275; visual cylinder length=0.05 radius=0.0275
- added link left_front_link, mass 1; collision cylinder length=0.05 radius=0.0275; visual cylinder length=0.05 radius=0.0275
- added link right_back_link, mass 1; collision cylinder length=0.05 radius=0.0275; visual cylinder length=0.05 radius=0.0275
- added link right_front_link, mass 1; collision cylinder length=0.05 radius=0.0275; visual cylinder length=0.05 radius=0.0275
- link left0_link: geometry collision cylinder length=0.05 radius=0.015; visual cylinder length=0.05 radius=0.015
- link left5_link: geometry collision cylinder length=0.05 radius=0.015; visual cylinder length=0.05 radius=0.015
- link right0_link: geometry collision cylinder length=0.05 radius=0.015; visual cylinder length=0.05 radius=0.015
- link right5_link: geometry collision cylinder length=0.05 radius=0.015; visual cylinder length=0.05 radius=0.015
Joints:
- added joint left_back_joint: type continuous, parent base_link, child left_back_link, origin xyz=-0.125 -0.095 -0.005 rpy=0 0 0, axis 0 1 0
- added joint left_front_joint: type continuous, parent base_link, child left_front_link, origin xyz=0.14 -0.095 -0.005 rpy=0 0 0, axis 0 1 0
- added joint right_back_joint: type continuous, parent base_link, child right_back_link, origin xyz=-0.125 0.095 -0.005 rpy=0 0 0, axis 0 1 0
- added joint right_front_joint: type continuous, parent base_link, child right_front_link, origin xyz=0.14 0.095 -0.005 rpy=0 0 0, axis 0 1 0
- joint left0_joint: origin xyz=0.14 -0.095 -0.005 rpy=0 0 0 -> xyz=0.14 -0.095 -0.05 rpy=0 0 0
- joint left5_joint: origin xyz=-0.125 -0.095 -0.005 rpy=0 0 0 -> xyz=-0.125 -0.095 -0.05 rpy=0 0 0
- joint right0_joint: origin xyz=0.14 0.095 -0.005 rpy=0 0 0 -> xyz=0.14 0.095 -0.05 rpy=0 0 0
- joint right5_joint: origin xyz=-0.125 0.095 -0.005 rpy=0 0 0 -> xyz=-0.125 0.095 -0.05 rpy=0 0 0

Commit message: add d435i model failed

File: src/caterpillar_robot/urdf/caterpillar_robot.xacro (robot description, xacro)
@@ -1,4 +1,6 @@
 <?xml version="1.0"?>
 <robot name="mycar" xmlns:xacro="http://wiki.ros.org/xacro">
+    <xacro:arg name="use_nominal_extrinsics" default="false" />
+    <xacro:include filename="$(find realsense2_description)/urdf/_d435i.urdf.xacro" />
     <xacro:property name="PI" value="3.1415926"/>
     <xacro:macro name="default_inertial" params="mass">
@@ -124,5 +126,5 @@
         <xacro:default_inertial mass="0.01"/>
     </link>
-    <link name="camera_link">
+    <!-- <link name="camera_link">
         <visual>
             <origin xyz="0 0 0" rpy="0 0 0"/>
@@ -144,5 +146,8 @@
         </collision>
         <xacro:default_inertial mass="0.01"/>
-    </link>
+    </link> -->
+    <xacro:sensor_d435i parent="tripod_link" use_nominal_extrinsics="$(arg use_nominal_extrinsics)">
+        <origin xyz="0 0 0.06" rpy="0 0 0" />
+    </xacro:sensor_d435i>
     <joint name="base_joint" type="fixed">
         <parent link="base_footprint"/>
@@ -165,9 +170,9 @@
         <origin xyz="-0.03 0.0 0.08" rpy="0 0 0"/>
     </joint>
-    <joint name="camera_joint" type="continuous">
+    <!-- <joint name="camera_joint" type="continuous">
         <parent link="tripod_link"/>
         <child link="camera_link"/>
         <origin xyz="0 0.0 0.06" rpy="0 0 0"/>
-    </joint>
+    </joint> -->
     <xacro:wheel_func wheel_name="left_front" xyz="0.14 -0.095 -0.005" rpy="0 0 0" radius="0.0275" length="0.05" mu="1" mu2="1"/>
     <xacro:wheel_func wheel_name="left0" xyz="0.14 -0.095 -0.05" rpy="0 0 0" radius="0.015" length="0.05" mu="1" mu2="1"/>

File: src/caterpillar_robot/urdf/caterpillar_robot.xacro.urdf (robot description, URDF)
Before this commit: robot mycar, 22 links, 21 joints
Links:
- added link camera_bottom_screw_frame
- link camera_link: mass 1 -> 0.072; geometry collision box size=0.02505 0.09 0.025; visual mesh filename=package://realsense2_description/meshes/d435.dae
Joints:
- added joint camera_link_joint: type fixed, parent camera_bottom_screw_frame, child camera_link, origin xyz=0.010600000000000002 0.0175 0.0125 rpy=0 0 0
- joint camera_joint: child camera_link -> camera_bottom_screw_frame; origin xyz=0 0.0 0.06 rpy=0 0 0 -> xyz=0 0 0.06 rpy=0 0 0; type continuous -> fixed

Commit message: git clone https://github.com/pal-robotics/realsense_gazebo_plugin.git -b foxy-devel git clone https://github.com/IntelligentSystemsLabUTV/realsense_ros2_gazebo.git

File: src/caterpillar_robot/urdf/caterpillar_robot.xacro (robot description, xacro)
@@ -1,6 +1,4 @@
 <?xml version="1.0"?>
 <robot name="mycar" xmlns:xacro="http://wiki.ros.org/xacro">
-    <xacro:arg name="use_nominal_extrinsics" default="false" />
-    <xacro:include filename="$(find realsense2_description)/urdf/_d435i.urdf.xacro" />
     <xacro:property name="PI" value="3.1415926"/>
     <xacro:macro name="default_inertial" params="mass">
@@ -147,7 +145,8 @@
         <xacro:default_inertial mass="0.01"/>
     </link> -->
-    <xacro:sensor_d435i parent="tripod_link" use_nominal_extrinsics="$(arg use_nominal_extrinsics)">
-        <origin xyz="0 0 0.06" rpy="0 0 0" />
-    </xacro:sensor_d435i>
+    <xacro:include filename="$(find realsense_ros2_gazebo)/xacro/depthcam.xacro"/>
+    <xacro:realsense_d435 sensor_name="d435" parent_link="tripod_link" rate="30">
+    <origin rpy="0 0 0 " xyz="0 0 0.045"/>
+    </xacro:realsense_d435>
     <joint name="base_joint" type="fixed">
         <parent link="base_footprint"/>
@@ -205,7 +204,7 @@
         <material>Gazebo/Gray</material>
     </gazebo>
-    <gazebo reference="camera_link">
+    <!-- <gazebo reference="camera_link">
         <material>Gazebo/Gray</material>
-    </gazebo>
+    </gazebo> -->
     <!-- <link name="caster_link">
       <visual>

File: src/caterpillar_robot/urdf/caterpillar_robot.xacro.urdf (robot description, URDF)
Before this commit: robot mycar, 23 links, 22 joints
Links:
- removed link camera_bottom_screw_frame
- removed link camera_link
- added link d435_bottom_screw_frame
- added link d435_color_frame
- added link d435_color_optical_frame
- added link d435_depth_frame
- added link d435_depth_optical_frame
- added link d435_left_ir_frame
- added link d435_left_ir_optical_frame
- added link d435_link, mass 0.564; collision box size=0.02505 0.09 0.025; visual mesh filename=file:///home/dillon/project/realsense_ros2_gazebo/install/r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
- added link d435_right_ir_frame
- added link d435_right_ir_optical_frame
Joints:
- removed joint camera_joint
- removed joint camera_link_joint
- added joint d435_color_joint: type fixed, parent d435_depth_frame, child d435_color_frame, origin xyz=0 0.015 0 rpy=0 0 0
- added joint d435_color_optical_joint: type fixed, parent d435_color_frame, child d435_color_optical_frame, origin xyz=0 0 0 rpy=-1.5707963267948966 0 -1.5707963267948966
- added joint d435_depth_joint: type fixed, parent d435_link, child d435_depth_frame, origin xyz=0 0 0 rpy=0 0 0
- added joint d435_depth_optical_joint: type fixed, parent d435_depth_frame, child d435_depth_optical_frame, origin xyz=0 0 0 rpy=-1.5707963267948966 0 -1.5707963267948966
- added joint d435_joint: type fixed, parent tripod_link, child d435_bottom_screw_frame, origin xyz=0 0 0.045 rpy=0 0 0 
- added joint d435_left_ir_joint: type fixed, parent d435_depth_frame, child d435_left_ir_frame, origin xyz=0 0.0 0 rpy=0 0 0
- added joint d435_left_ir_optical_joint: type fixed, parent d435_left_ir_frame, child d435_left_ir_optical_frame, origin xyz=0 0 0 rpy=-1.5707963267948966 0 -1.5707963267948966
- added joint d435_link_joint: type fixed, parent d435_bottom_screw_frame, child d435_link, origin xyz=0 0.0175 0.0125 rpy=0 0 0
- added joint d435_right_ir_joint: type fixed, parent d435_depth_frame, child d435_right_ir_frame, origin xyz=0 -0.05 0 rpy=0 0 0
- added joint d435_right_ir_optical_joint: type fixed, parent d435_right_ir_frame, child d435_right_ir_optical_frame, origin xyz=0 0 0 rpy=-1.5707963267948966 0 -1.5707963267948966
