Commit message: fix model file, add MUV function and .......fuck you CSDN

File: src/caterpillar_robot/urdf/caterpillar_robot.xacro (robot description, xacro)
@@ -1,4 +1,6 @@
 <?xml version="1.0"?>
-<robot name="mycar" xmlns:xacro="http://wiki.ros.org/xacro">
+<robot name="robot" xmlns:xacro="http://wiki.ros.org/xacro">
+    <!-- <xacro:arg name="ns" default="" /> -->
+    <xacro:property name="robot_name" value="$(arg ns)"/>
     <xacro:property name="PI" value="3.1415926"/>
     <xacro:macro name="default_inertial" params="mass">
@@ -9,5 +11,5 @@
 	</xacro:macro>
     <xacro:macro name="wheel_func" params="wheel_name radius length xyz rpy mu mu2" >
-        <link name="${wheel_name}_link">
+        <link name="${robot_name}_${wheel_name}_link">
             <visual>
                 <geometry>
@@ -21,24 +23,19 @@
                     <cylinder radius="${radius}" length="${length}" />
                 </geometry>
-                <!-- <surface>
-                    <friction>
-                        <ode mu="${mu}" mu2="${mu2}"/>
-                    </friction>
-                </surface> -->
             </collision>
             <xacro:default_inertial mass="0.3"/>
         </link>
-        <joint name="${wheel_name}_joint" type="continuous">
-            <parent link="base_link"/>
-            <child link="${wheel_name}_link"/>
+        <joint name="${robot_name}_${wheel_name}_joint" type="continuous">
+            <parent link="${robot_name}_base_link"/>
+            <child link="${robot_name}_${wheel_name}_link"/>
             <origin xyz="${xyz}" rpy="${rpy}"/>
             <axis xyz="0 1 0" />
         </joint>
-        <gazebo reference="${wheel_name}_link">
+        <gazebo reference="${robot_name}_${wheel_name}_link">
             <material>Gazebo/Gray</material>
         </gazebo>
     </xacro:macro>
-    <link name="base_footprint"/>
-    <link name="base_link">
+    <link name="${robot_name}_base_footprint"/>
+    <link name="${robot_name}_base_link">
         <visual>
             <origin xyz="0 0 0" rpy="0 0 0"/>
@@ -61,5 +58,5 @@
         <xacro:default_inertial mass="2"/>
     </link>
-    <link name="plat_link">
+    <link name="${robot_name}_plat_link">
         <visual>
             <origin xyz="0 0 0.0" rpy="0 0 0"/>
@@ -82,5 +79,5 @@
         <xacro:default_inertial mass="0.02"/>
     </link>
-    <link name="laser_link">
+    <link name="${robot_name}_laser_link">
         <visual>
             <origin xyz="0 0 0" rpy="0 0 0"/>
@@ -103,5 +100,5 @@
         <xacro:default_inertial mass="0.01"/>
     </link>
-    <link name="tripod_link">
+    <link name="${robot_name}_tripod_link">
         <visual>
             <origin xyz="0 0 0" rpy="0 0 0"/>
@@ -124,54 +121,28 @@
         <xacro:default_inertial mass="0.01"/>
     </link>
-    <!-- <link name="camera_link">
-        <visual>
-            <origin xyz="0 0 0" rpy="0 0 0"/>
-            <geometry>
-                <box size="0.025 0.09 0.03"/>
-            </geometry>
-            <material name="black">
-                <color rgba="0.0 0.0 0.0 0.5" />
-            </material>
-        </visual>
-        <collision>
-            <origin xyz="0 0 0" rpy="0 0 0"/>
-            <geometry>
-                <box size="0.025 0.09 0.03"/>
-            </geometry>
-                <material name="black">
-                <color rgba="0.0 0.0 0.0 0.5" />
-            </material>
-        </collision>
-        <xacro:default_inertial mass="0.01"/>
-    </link> -->
-    <xacro:include filename="$(find realsense_ros2_gazebo)/xacro/depthcam.xacro"/>
+    <!-- <xacro:include filename="$(find realsense_ros2_gazebo)/xacro/depthcam.xacro"/>
     <xacro:realsense_d435 sensor_name="d435" parent_link="tripod_link" rate="30">
     <origin rpy="0 0 0 " xyz="0 0 0.045"/>
-    </xacro:realsense_d435>
-    <joint name="base_joint" type="fixed">
-        <parent link="base_footprint"/>
-        <child link="base_link"/>
+    </xacro:realsense_d435> -->
+    <joint name="${robot_name}_base_joint" type="fixed">
+        <parent link="${robot_name}_base_footprint"/>
+        <child link="${robot_name}_base_link"/>
         <origin xyz="0.0 0.0 0.1" rpy="0 0 0"/>
     </joint>
-    <joint name="plat_joint" type="fixed">
-        <parent link="base_link"/>
-        <child link="plat_link"/>
+    <joint name="${robot_name}_plat_joint" type="fixed">
+        <parent link="${robot_name}_base_link"/>
+        <child link="${robot_name}_plat_link"/>
         <origin xyz="-0.055 0.0 0.07" rpy="0 0 0"/>
     </joint>
-    <joint name="laser_joint" type="fixed">
-        <parent link="plat_link"/>
-        <child link="laser_link"/>
+    <joint name="${robot_name}_laser_joint" type="fixed">
+        <parent link="${robot_name}_plat_link"/>
+        <child link="${robot_name}_laser_link"/>
         <origin xyz="0.055 0.0 0.05" rpy="0 0 0"/>
     </joint>
-    <joint name="tripod_joint" type="fixed">
-        <parent link="plat_link"/>
-        <child link="tripod_link"/>
+    <joint name="${robot_name}_tripod_joint" type="fixed">
+        <parent link="${robot_name}_plat_link"/>
+        <child link="${robot_name}_tripod_link"/>
         <origin xyz="-0.03 0.0 0.08" rpy="0 0 0"/>
     </joint>
-    <!-- <joint name="camera_joint" type="continuous">
-        <parent link="tripod_link"/>
-        <child link="camera_link"/>
-        <origin xyz="0 0.0 0.06" rpy="0 0 0"/>
-    </joint> -->
     <xacro:wheel_func wheel_name="left_front" xyz="0.14 -0.095 -0.005" rpy="0 0 0" radius="0.0275" length="0.05" mu="1" mu2="1"/>
     <xacro:wheel_func wheel_name="left0" xyz="0.14 -0.095 -0.05" rpy="0 0 0" radius="0.015" length="0.05" mu="1" mu2="1"/>
@@ -182,5 +153,4 @@
     <xacro:wheel_func wheel_name="left5" xyz="-0.125 -0.095 -0.05" rpy="0 0 0" radius="0.015" length="0.05" mu="1" mu2="1"/>
     <xacro:wheel_func wheel_name="left_back" xyz="-0.125 -0.095 -0.005" rpy="0 0 0" radius="0.0275" length="0.05" mu="1" mu2="1"/>
-    <!-- <xacro:wheel_func wheel_name="leftv" xyz="-0.1 -0.15 -0.04" rpy="0 0 0" radius="0.0275" length="0.05" mu="4" mu2="4"/> -->
     <xacro:wheel_func wheel_name="right_front" xyz="0.14 0.095 -0.005" rpy="0 0 0" radius="0.0275" length="0.05" mu="1" mu2="1"/>
     <xacro:wheel_func wheel_name="right0" xyz="0.14 0.095 -0.05" rpy="0 0 0" radius="0.015" length="0.05" mu="1" mu2="1"/>
@@ -191,71 +161,44 @@
     <xacro:wheel_func wheel_name="right5" xyz="-0.125 0.095 -0.05" rpy="0 0 0" radius="0.015" length="0.05" mu="1" mu2="1"/>
     <xacro:wheel_func wheel_name="right_back" xyz="-0.125 0.095 -0.005" rpy="0 0 0" radius="0.0275" length="0.05" mu="1" mu2="1"/>
-    <!-- <xacro:wheel_func wheel_name="rightv" xyz="-0.1 0.15 -0.04" rpy="0 0 0" radius="0.0275" length="0.05" mu="4" mu2="4"/> -->
-    <gazebo reference="base_link">
+    <gazebo reference="${robot_name}_base_link">
         <material>Gazebo/Green</material>
     </gazebo>
-    <gazebo reference="plat_link">
+    <gazebo reference="${robot_name}_plat_link">
         <material>Gazebo/Black</material>
     </gazebo>
-    <gazebo reference="laser_link">
+    <gazebo reference="${robot_name}_laser_link">
         <material>Gazebo/Gray</material>
     </gazebo>
-    <gazebo reference="tripod_link">
+    <gazebo reference="${robot_name}_tripod_link">
         <material>Gazebo/Gray</material>
     </gazebo>
-    <!-- <gazebo reference="camera_link">
-        <material>Gazebo/Gray</material>
-    </gazebo> -->
-    <!-- <link name="caster_link">
-      <visual>
-        <origin xyz="0 0 0" rpy="1.57079 0 0"/>
-        <geometry>
-            <sphere radius="0.015"/>
-        </geometry>
-          <material name="black">
-            <color rgba="0.0 0.0 0.0 0.5" />
-          </material>
-      </visual>
-      <collision>
-        <origin xyz="0 0 0" rpy="1.57079 0 0"/>
-        <geometry>
-            <sphere radius="0.015"/>
-        </geometry>
-          <material name="black">
-            <color rgba="0.0 0.0 0.0 0.5" />
-          </material>
-          <surface>
-            <friction>
-                <ode mu="0" mu2="0"/>
-            </friction>
-        </surface>
-      </collision>
-      <xacro:default_inertial mass="0.3"/>
-  </link>
-  <joint name="caster_joint" type="fixed">
-      <parent link="base_link" />
-      <child link="caster_link" />
-      <origin xyz="0.15 0.0 -0.05" />
-      <axis xyz="0 1 0" />
-  </joint> -->
     <gazebo>
-        <plugin name='diff_drive' filename='libgazebo_ros_planar_move.so'>
-            <leftFrontJoint>left0_joint</leftFrontJoint>
-			<rightFrontJoint>right0_joint</rightFrontJoint>
-			<leftRearJoint>left5_joint</leftRearJoint>
-			<rightRearJoint>right5_joint</rightRearJoint>
-            <commandTopic>cmd_vel</commandTopic>
-			<odometryTopic>odom</odometryTopic>
-			<odometryFrame>odom</odometryFrame>
-			<robotNamespace>/</robotNamespace>
+        <plugin name='${robot_name}_diff_drive' filename='libgazebo_ros_planar_move.so'>
+            <ros>
+                <namespace>/${robot_name}</namespace>
+            </ros>
+            <update_rate>100</update_rate>
+            <publish_rate>10</publish_rate>
+            <publish_odom>true</publish_odom>
+            <publish_odom_tf>true</publish_odom_tf>
+            <odometry_frame>${robot_name}_odom</odometry_frame>
+            <robot_base_frame>${robot_name}_base_footprint</robot_base_frame>
+            <!-- <leftFrontJoint>${robot_name}_left0_joint</leftFrontJoint>
+			<rightFrontJoint>${robot_name}_right0_joint</rightFrontJoint>
+			<leftRearJoint>${robot_name}_left5_joint</leftRearJoint>
+			<rightRearJoint>${robot_name}_right5_joint</rightRearJoint>
+            <commandTopic>/${robot_name}/cmd_vel</commandTopic>
+			<odometryTopic>/${robot_name}/odom</odometryTopic>
+			<odometryFrame>${robot_name}_odom</odometryFrame>
 			<odometryRate>10.0</odometryRate>
             <publish_odom>true</publish_odom>
             <publish_odom_tf>true</publish_odom_tf>
             <publish_wheel_tf>true</publish_wheel_tf>
-			<robotBaseFrame>base_footprint</robotBaseFrame>
+			<robotBaseFrame>${robot_name}_base_footprint</robotBaseFrame>
+            <broadcastTF>1</broadcastTF> -->
         </plugin>
     </gazebo>
-    <gazebo reference="laser_link">
-        <sensor name="laser_sensor" type="ray">
+    <gazebo reference="${robot_name}_laser_link">
+        <sensor name="${robot_name}_laser_sensor" type="ray">
         <always_on>true</always_on>
         <visualize>false</visualize>
@@ -267,6 +210,4 @@
                 <samples>360</samples>
                 <resolution>1.000000</resolution>
-                <!-- <min_angle>-2.3561944901923449288469825374596</min_angle>
-                <max_angle>2.3561944901923449288469825374596</max_angle> -->
                 <min_angle>0.00</min_angle>
                 <max_angle>6.28</max_angle>
@@ -284,7 +225,8 @@
             </noise>
         </ray>
-        <plugin name="laserscan" filename="libgazebo_ros_ray_sensor.so">
+        <plugin name="${robot_name}_laserscan" filename="libgazebo_ros_ray_sensor.so">
+          <robotNamespace>/${robot_name}</robotNamespace>
           <ros>
-            <!-- <namespace>/tb3</namespace> -->
+            <namespace>/${robot_name}</namespace>
             <remapping>~/out:=scan</remapping>
           </ros>

Commit message: mav planning ok

File: src/caterpillar_robot/urdf/caterpillar_robot.xacro (robot description, xacro)
@@ -1,6 +1,10 @@
 <?xml version="1.0"?>
 <robot name="robot" xmlns:xacro="http://wiki.ros.org/xacro">
-    <!-- <xacro:arg name="ns" default="" /> -->
-    <xacro:property name="robot_name" value="$(arg ns)"/>
+    <xacro:arg name="robot_color" default="Green" />
+    <xacro:arg name="robot_name" default="robot" />
+    <xacro:arg name="robot_namespace" default="" />
+    <xacro:property name="robot_color" value="$(arg robot_color)"/>
+    <xacro:property name="robot_name" value="$(arg robot_name)"/>
+    <xacro:property name="robot_namespace" value="$(arg robot_namespace)"/>
     <xacro:property name="PI" value="3.1415926"/>
     <xacro:macro name="default_inertial" params="mass">
@@ -121,5 +125,5 @@
         <xacro:default_inertial mass="0.01"/>
     </link>
-    <xacro:include filename="$(find realsense_ros2_gazebo)/xacro/d435.xacro"/>
+    <xacro:include filename="$(find caterpillar_robot)/urdf/d435.xacro"/>
     <xacro:realsense_d435 sensor_name="${robot_name}_d435" parent_link="${robot_name}_tripod_link" rate="30" robot_name="${robot_name}">
     <origin rpy="0 0 0 " xyz="0 0 0.045"/>
@@ -162,5 +166,5 @@
     <xacro:wheel_func wheel_name="right_back" xyz="-0.125 0.095 -0.005" rpy="0 0 0" radius="0.0275" length="0.05" mu="1" mu2="1"/>
     <gazebo reference="${robot_name}_base_link">
-        <material>Gazebo/Green</material>
+        <material>Gazebo/${robot_color}</material>
     </gazebo>
     <gazebo reference="${robot_name}_plat_link">
@@ -176,25 +180,12 @@
         <plugin name='${robot_name}_diff_drive' filename='libgazebo_ros_planar_move.so'>
             <ros>
-                <namespace>/${robot_name}</namespace>
+                <namespace>/${robot_namespace}</namespace>
             </ros>
             <update_rate>100</update_rate>
-            <publish_rate>10</publish_rate>
+            <publish_rate>100</publish_rate>
             <publish_odom>true</publish_odom>
             <publish_odom_tf>true</publish_odom_tf>
             <odometry_frame>${robot_name}_odom</odometry_frame>
             <robot_base_frame>${robot_name}_base_footprint</robot_base_frame>
-            <!-- <leftFrontJoint>${robot_name}_left0_joint</leftFrontJoint>
-			<rightFrontJoint>${robot_name}_right0_joint</rightFrontJoint>
-			<leftRearJoint>${robot_name}_left5_joint</leftRearJoint>
-			<rightRearJoint>${robot_name}_right5_joint</rightRearJoint>
-            <commandTopic>/${robot_name}/cmd_vel</commandTopic>
-			<odometryTopic>/${robot_name}/odom</odometryTopic>
-			<odometryFrame>${robot_name}_odom</odometryFrame>
-			<odometryRate>10.0</odometryRate>
-            <publish_odom>true</publish_odom>
-            <publish_odom_tf>true</publish_odom_tf>
-            <publish_wheel_tf>true</publish_wheel_tf>
-			<robotBaseFrame>${robot_name}_base_footprint</robotBaseFrame>
-            <broadcastTF>1</broadcastTF> -->
         </plugin>
     </gazebo>
@@ -226,7 +217,7 @@
         </ray>
         <plugin name="${robot_name}_laserscan" filename="libgazebo_ros_ray_sensor.so">
-          <robotNamespace>/${robot_name}</robotNamespace>
+          <robotNamespace>/${robot_namespace}</robotNamespace>
           <ros>
-            <namespace>/${robot_name}</namespace>
+            <namespace>/${robot_namespace}</namespace>
             <remapping>~/out:=scan</remapping>
           </ros>

File: src/caterpillar_robot/urdf/caterpillar_robot_withoutsensor.xacro (robot description, xacro)
@@ -1,6 +1,10 @@
 <?xml version="1.0"?>
 <robot name="robot" xmlns:xacro="http://wiki.ros.org/xacro">
-    <!-- <xacro:arg name="ns" default="" /> -->
-    <xacro:property name="robot_name" value="$(arg ns)"/>
+    <xacro:arg name="robot_color" default="Green" />
+    <xacro:arg name="robot_name" default="robot" />
+    <xacro:arg name="robot_namespace" default="" />
+    <xacro:property name="robot_color" value="$(arg robot_color)"/>
+    <xacro:property name="robot_name" value="$(arg robot_name)"/>
+    <xacro:property name="robot_namespace" value="$(arg robot_namespace)"/>
     <xacro:property name="PI" value="3.1415926"/>
     <xacro:macro name="default_inertial" params="mass">
@@ -141,22 +145,22 @@
         <origin xyz="-0.03 0.0 0.08" rpy="0 0 0"/>
     </joint>
-    <!-- <xacro:wheel_func wheel_name="left_front" xyz="0.14 -0.095 -0.005" rpy="0 0 0" radius="0.0275" length="0.05" mu="1" mu2="1"/> -->
+    <xacro:wheel_func wheel_name="left_front" xyz="0.14 -0.095 -0.005" rpy="0 0 0" radius="0.0275" length="0.05" mu="1" mu2="1"/>
     <xacro:wheel_func wheel_name="left0" xyz="0.14 -0.095 -0.05" rpy="0 0 0" radius="0.015" length="0.05" mu="1" mu2="1"/>
-    <!-- <xacro:wheel_func wheel_name="left1" xyz="0.075 -0.095 -0.05" rpy="0 0 0" radius="0.015" length="0.05" mu="1" mu2="1"/>
+    <xacro:wheel_func wheel_name="left1" xyz="0.075 -0.095 -0.05" rpy="0 0 0" radius="0.015" length="0.05" mu="1" mu2="1"/>
     <xacro:wheel_func wheel_name="left2" xyz="0.025 -0.095 -0.05" rpy="0 0 0" radius="0.015" length="0.05" mu="1" mu2="1"/>
     <xacro:wheel_func wheel_name="left3" xyz="-0.025 -0.095 -0.05" rpy="0 0 0" radius="0.015" length="0.05" mu="1" mu2="1"/>
-    <xacro:wheel_func wheel_name="left4" xyz="-0.075 -0.095 -0.05" rpy="0 0 0" radius="0.015" length="0.05" mu="1" mu2="1"/> -->
+    <xacro:wheel_func wheel_name="left4" xyz="-0.075 -0.095 -0.05" rpy="0 0 0" radius="0.015" length="0.05" mu="1" mu2="1"/>
     <xacro:wheel_func wheel_name="left5" xyz="-0.125 -0.095 -0.05" rpy="0 0 0" radius="0.015" length="0.05" mu="1" mu2="1"/>
-    <!-- <xacro:wheel_func wheel_name="left_back" xyz="-0.125 -0.095 -0.005" rpy="0 0 0" radius="0.0275" length="0.05" mu="1" mu2="1"/>
-    <xacro:wheel_func wheel_name="right_front" xyz="0.14 0.095 -0.005" rpy="0 0 0" radius="0.0275" length="0.05" mu="1" mu2="1"/> -->
+    <xacro:wheel_func wheel_name="left_back" xyz="-0.125 -0.095 -0.005" rpy="0 0 0" radius="0.0275" length="0.05" mu="1" mu2="1"/>
+    <xacro:wheel_func wheel_name="right_front" xyz="0.14 0.095 -0.005" rpy="0 0 0" radius="0.0275" length="0.05" mu="1" mu2="1"/>
     <xacro:wheel_func wheel_name="right0" xyz="0.14 0.095 -0.05" rpy="0 0 0" radius="0.015" length="0.05" mu="1" mu2="1"/>
-    <!-- <xacro:wheel_func wheel_name="right1" xyz="0.075 0.095 -0.05" rpy="0 0 0" radius="0.015" length="0.05" mu="1" mu2="1"/>
+    <xacro:wheel_func wheel_name="right1" xyz="0.075 0.095 -0.05" rpy="0 0 0" radius="0.015" length="0.05" mu="1" mu2="1"/>
     <xacro:wheel_func wheel_name="right2" xyz="0.025 0.095 -0.05" rpy="0 0 0" radius="0.015" length="0.05" mu="1" mu2="1"/>
     <xacro:wheel_func wheel_name="right3" xyz="-0.025 0.095 -0.05" rpy="0 0 0" radius="0.015" length="0.05" mu="1" mu2="1"/>
-    <xacro:wheel_func wheel_name="right4" xyz="-0.075 0.095 -0.05" rpy="0 0 0" radius="0.015" length="0.05" mu="1" mu2="1"/> -->
+    <xacro:wheel_func wheel_name="right4" xyz="-0.075 0.095 -0.05" rpy="0 0 0" radius="0.015" length="0.05" mu="1" mu2="1"/>
     <xacro:wheel_func wheel_name="right5" xyz="-0.125 0.095 -0.05" rpy="0 0 0" radius="0.015" length="0.05" mu="1" mu2="1"/>
-    <!-- <xacro:wheel_func wheel_name="right_back" xyz="-0.125 0.095 -0.005" rpy="0 0 0" radius="0.0275" length="0.05" mu="1" mu2="1"/> -->
+    <xacro:wheel_func wheel_name="right_back" xyz="-0.125 0.095 -0.005" rpy="0 0 0" radius="0.0275" length="0.05" mu="1" mu2="1"/>
     <gazebo reference="${robot_name}_base_link">
-        <material>Gazebo/Green</material>
+        <material>Gazebo/${robot_color}</material>
     </gazebo>
     <gazebo reference="${robot_name}_plat_link">
@@ -172,7 +176,7 @@
         <plugin name='${robot_name}_diff_drive' filename='libgazebo_ros_planar_move.so'>
             <ros>
-                <namespace>/${robot_name}</namespace>
+                <namespace>/${robot_namespace}</namespace>
             </ros>
-            <update_rate>10</update_rate>
+            <update_rate>100</update_rate>
             <publish_rate>10</publish_rate>
             <publish_odom>true</publish_odom>
@@ -180,17 +184,4 @@
             <odometry_frame>${robot_name}_odom</odometry_frame>
             <robot_base_frame>${robot_name}_base_footprint</robot_base_frame>
-            <!-- <leftFrontJoint>${robot_name}_left0_joint</leftFrontJoint>
-			<rightFrontJoint>${robot_name}_right0_joint</rightFrontJoint>
-			<leftRearJoint>${robot_name}_left5_joint</leftRearJoint>
-			<rightRearJoint>${robot_name}_right5_joint</rightRearJoint>
-            <commandTopic>/${robot_name}/cmd_vel</commandTopic>
-			<odometryTopic>/${robot_name}/odom</odometryTopic>
-			<odometryFrame>${robot_name}_odom</odometryFrame>
-			<odometryRate>10.0</odometryRate>
-            <publish_odom>true</publish_odom>
-            <publish_odom_tf>true</publish_odom_tf>
-            <publish_wheel_tf>true</publish_wheel_tf>
-			<robotBaseFrame>${robot_name}_base_footprint</robotBaseFrame>
-            <broadcastTF>1</broadcastTF> -->
         </plugin>
     </gazebo>

Commit message: try to set jointstate failed

File: src/caterpillar_robot/urdf/caterpillar_robot.xacro (robot description, xacro)
@@ -144,8 +144,10 @@
         <origin xyz="0.055 0.0 0.05" rpy="0 0 0"/>
     </joint>
-    <joint name="${robot_name}_tripod_joint" type="fixed">
+    <joint name="${robot_name}_tripod_joint" type="revolute">
         <parent link="${robot_name}_plat_link"/>
         <child link="${robot_name}_tripod_link"/>
         <origin xyz="-0.03 0.0 0.08" rpy="0 0 0"/>
+        <axis xyz="0 0 1" />
+        <limit effort="30" velocity="1.0" lower="-2.3561944" upper="2.3561944" />
     </joint>
     <xacro:wheel_func wheel_name="left_front" xyz="0.14 -0.095 -0.005" rpy="0 0 0" radius="0.0275" length="0.05" mu="1" mu2="1"/>
@@ -227,3 +229,12 @@
         </sensor>
       </gazebo>
+    <gazebo>
+        <plugin name="${robot_name}_tripod_trajectory" filename="libgazebo_ros_joint_pose_trajectory.so">
+            <ros>
+                <namespace>/${robot_namespace}</namespace>
+                <!-- <remapping>set_joint_trajectory:=tripod</remapping> -->
+            </ros>
+            <update_rate>2</update_rate>
+        </plugin>
+    </gazebo>
 </robot>

Commit message: add arm xacro

File: src/caterpillar_robot/urdf/caterpillar_robot.xacro (robot description, xacro)
@@ -125,8 +125,4 @@
         <xacro:default_inertial mass="0.01"/>
     </link>
-    <xacro:include filename="$(find caterpillar_robot)/urdf/d435.xacro"/>
-    <xacro:realsense_d435 sensor_name="${robot_name}_d435" parent_link="${robot_name}_tripod_link" rate="30" robot_name="${robot_name}">
-    <origin rpy="0 0 0 " xyz="0 0 0.045"/>
-    </xacro:realsense_d435>
     <joint name="${robot_name}_base_joint" type="fixed">
         <parent link="${robot_name}_base_footprint"/>
@@ -179,4 +175,12 @@
         <material>Gazebo/Gray</material>
     </gazebo>
+    <xacro:include filename="$(find caterpillar_robot)/urdf/d435.xacro"/>
+    <xacro:realsense_d435 sensor_name="${robot_name}_d435" parent_link="${robot_name}_tripod_link" rate="30" robot_name="${robot_name}">
+        <origin rpy="0 0 0 " xyz="0 0 0.045"/>
+    </xacro:realsense_d435>
+    <xacro:include filename="$(find caterpillar_robot)/urdf/servo_arm.xacro"/>
+    <xacro:servo_arm robot_name="${robot_name}" arm_name="arm" parent_link="${robot_name}_base_link">
+        <origin rpy="0 0 0 " xyz="0.2 0 0"/>
+    </xacro:servo_arm>
     <gazebo>
         <plugin name='${robot_name}_diff_drive' filename='libgazebo_ros_planar_move.so'>
