Commit message: fix servo plugin and add servoarm ok

File: src/caterpillar_robot/urdf/caterpillar_robot.xacro (robot description, xacro)
@@ -138,5 +138,5 @@
         <parent link="${robot_name}_plat_link"/>
         <child link="${robot_name}_laser_link"/>
-        <origin xyz="0.055 0.0 0.05" rpy="0 0 0"/>
+        <origin xyz="0.055 0.0 0.08" rpy="0 0 0"/>
     </joint>
     <joint name="${robot_name}_tripod_joint" type="revolute">
@@ -181,5 +181,5 @@
     <xacro:include filename="$(find caterpillar_robot)/urdf/servo_arm.xacro"/>
     <xacro:servo_arm robot_name="${robot_name}" arm_name="arm" parent_link="${robot_name}_base_link">
-        <origin rpy="0 0 0 " xyz="0.2 0 0"/>
+        <origin rpy="0 0 0 " xyz="0.15 0 -0.01"/>
     </xacro:servo_arm>
     <gazebo>
@@ -237,5 +237,5 @@
             <ros>
                 <namespace>/${robot_namespace}</namespace>
-                <!-- <remapping>set_joint_trajectory:=tripod</remapping> -->
+                <remapping>set_servojoint:=tripod</remapping>
             </ros>
             <update_rate>10</update_rate>

File: src/caterpillar_robot/urdf/servo_arm.xacro (robot description, xacro)
@@ -31,5 +31,5 @@
         <link name="${robot_name}_${arm_name}_arm_link">
             <visual>
-                <origin xyz="0 0 0" rpy="0 0 0"/>
+                <origin xyz="0.05 0 0" rpy="0 0 0"/>
                 <geometry>
                     <box size="0.100 0.020 0.02"/>
@@ -40,5 +40,5 @@
             </visual>
             <collision>
-                <origin xyz="0 0 0" rpy="0 0 0"/>
+                <origin xyz="0.05 0 0" rpy="0 0 0"/>
                 <geometry>
                     <box size="0.100 0.020 0.02"/>
@@ -52,7 +52,7 @@
         <link name="${robot_name}_${arm_name}_hand_link">
             <visual>
-                <origin xyz="0 0 0" rpy="0 0 0"/>
+                <origin xyz="0.025 0 0" rpy="0 0 0"/>
                 <geometry>
-                    <box size="0.100 0.020 0.02"/>
+                    <box size="0.05 0.020 0.02"/>
                 </geometry>
                 <material name="blue">
@@ -61,7 +61,7 @@
             </visual>
             <collision>
-                <origin xyz="0 0 0" rpy="0 0 0"/>
+                <origin xyz="0.025 0 0" rpy="0 0 0"/>
                 <geometry>
-                    <box size="0.100 0.020 0.02"/>
+                    <box size="0.05 0.020 0.02"/>
                 </geometry>
                 <material name="blue">
@@ -80,5 +80,5 @@
             <parent link="${robot_name}_${arm_name}_base_link"/>
             <child link="${robot_name}_${arm_name}_arm_link"/>
-            <origin xyz="0.1 0 0" rpy="0 0 0"/>
+            <origin xyz="0.05 0 0" rpy="0 0 0"/>
             <axis xyz="0 1 0" />
         </joint>
@@ -98,4 +98,24 @@
             <material>Gazebo/Turquoise</material>
         </gazebo>
+        <gazebo>
+            <plugin name="${robot_name}_${arm_name}_arm_trajectory" filename="libgazebo_ros_servojoint.so">
+                <ros>
+                    <namespace>/${robot_namespace}</namespace>
+                    <remapping>set_servojoint:=${arm_name}_arm</remapping>
+                </ros>
+                <update_rate>10</update_rate>
+                <joints>${robot_name}_${arm_name}_arm_joint</joints>
+            </plugin>
+        </gazebo>
+        <gazebo>
+            <plugin name="${robot_name}_${arm_name}_hand_trajectory" filename="libgazebo_ros_servojoint.so">
+                <ros>
+                    <namespace>/${robot_namespace}</namespace>
+                    <remapping>set_servojoint:=${arm_name}_hand</remapping>
+                </ros>
+                <update_rate>10</update_rate>
+                <joints>${robot_name}_${arm_name}_hand_joint</joints>
+            </plugin>
+        </gazebo>
     </xacro:macro>
 </robot>
