Commit message: fix arm

File: src/caterpillar_robot/urdf/servo_arm.xacro (robot description, xacro)
@@ -71,4 +71,25 @@
             <xacro:dummy_inertial mass="0.01"/>
         </link>
+        <link name="${robot_name}_${arm_name}_function">
+            <visual>
+                <origin xyz="0 0 0" rpy="0 0 0"/>
+                <geometry>
+                    <box size="0.005 0.2 0.02"/>
+                </geometry>
+                <material name="blue">
+                    <color rgba="0.1 0.1 1.0 0.5" />
+                </material>
+            </visual>
+            <collision>
+                <origin xyz="0 0 0" rpy="0 0 0"/>
+                <geometry>
+                    <box size="0.005 0.2 0.02"/>
+                </geometry>
+                <material name="blue">
+                    <color rgba="0.1 0.1 1.0 0.5" />
+                </material>
+            </collision>
+            <xacro:dummy_inertial mass="0.01"/>
+        </link>
         <joint name="${robot_name}_${arm_name}_base_joint" type="fixed">
             <xacro:insert_block name="origin" />
@@ -89,4 +110,9 @@
             <axis xyz="0 1 0" />
         </joint>
+        <joint name="${robot_name}_${arm_name}_function_joint" type="fixed">
+            <parent link="${robot_name}_${arm_name}_hand_link"/>
+            <child link="${robot_name}_${arm_name}_function"/>
+            <origin xyz="0.0525 0 0" rpy="0 0 0"/>
+        </joint>
         <gazebo reference="${robot_name}_${arm_name}_base_link">
             <material>Gazebo/Turquoise</material>
@@ -97,4 +123,7 @@
         <gazebo reference="${robot_name}_${arm_name}_hand_link">
             <material>Gazebo/Turquoise</material>
+        </gazebo>
+        <gazebo reference="${robot_name}_${arm_name}_function">
+            <material>Gazebo/Gray</material>
         </gazebo>
         <gazebo>
